File: templates/BeagleBone/BB-cape-mitered-0603.sch (EAGLE design)
At the start: 14 parts, among them IC8 EEPROM-I2CSMD

Commit message: changed pull-ups to srm recommended 5.6k
Parts:
- R11, R2, R3, R6, R7, R8: value 4.7k -> 5.6k
Changed lines of the file:
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@@
 <part name="U$3" library="logic-supply" deviceset="FRAME_A3" device=""/>
 <part name="U$4" library="logic-supply" deviceset="LOGO-LGX" device="_LARGE" value="LOGO-LGX_LARGE"/>
-<part name="R7" library="rcl" deviceset="R-US_" device="R0603" value="4.7k">
+<part name="R7" library="rcl" deviceset="R-US_" device="R0603" value="5.6k">
 <attribute name="PARTNO" value="RC0603FR-074K7L"/>
 </part>
-<part name="R11" library="rcl" deviceset="R-US_" device="R0603" value="4.7k">
+<part name="R11" library="rcl" deviceset="R-US_" device="R0603" value="5.6k">
 <attribute name="PARTNO" value="RC0603FR-074K7L"/>
 </part>
 <part name="P+6" library="SparkFun-Aesthetics" deviceset="3.3V" device=""/>
-<part name="R2" library="rcl" deviceset="R-US_" device="R0603" value="4.7k">
+<part name="R2" library="rcl" deviceset="R-US_" device="R0603" value="5.6k">
 <attribute name="PARTNO" value="RC0603FR-074K7L"/>
 </part>
 <part name="TP1" library="logic-supply" deviceset="TEST_POINT" device=""/>
 <part name="GND9" library="supply1" deviceset="GND" device=""/>
-<part name="R3" library="rcl" deviceset="R-US_" device="R0603" value="4.7k">
+<part name="R3" library="rcl" deviceset="R-US_" device="R0603" value="5.6k">
 <attribute name="PARTNO" value="RC0603FR-074K7L"/>
 </part>
-<part name="R6" library="rcl" deviceset="R-US_" device="R0603" value="4.7k">
+<part name="R6" library="rcl" deviceset="R-US_" device="R0603" value="5.6k">
 <attribute name="PARTNO" value="RC0603FR-074K7L"/>
 </part>
-<part name="R8" library="rcl" deviceset="R-US_" device="R0603" value="4.7k">
+<part name="R8" library="rcl" deviceset="R-US_" device="R0603" value="5.6k">
 <attribute name="PARTNO" value="RC0603FR-074K7L"/>
 </part>

Commit message: renumbered components on templates
Parts:
- removed R11: 5.6k, rcl:R-US_R0603
- added R4: 5.6k, rcl:R-US_R0603
- TP1: BOM (none) -> EXCLUDE
- TP2: BOM EXCLUDE -> (none)
- renumbered C13 to C1, IC8 to IC1, R7 to R5, R8 to R1, S3 to S1
Connections:
- net 3.3V: now also R4.2; no longer R11.2
- net GND: now also TP1.P$1; no longer TP2.P$1
- net I2C2_SDA: now also R6.1; no longer R11.1
- net N$14: now also R2.1; no longer R6.1
- net WP: now also R4.1, TP2.P$1; no longer R2.1, TP1.P$1
Other:
- moved on the sheet: R2, R6, TP1, TP2
